File: StepperTMC2240.kicad_sch (KiCad schematic)
At the start: 24 parts, among them J1 V_{MOTOR}, J4 Motor, Q1 Q_NMOS_GSD, U1 TMC2240_TQFN

Commit message: Added an ADC input pin, and protection diodes. Updated the OV load resistor to 0805. Cleaned up a few silk screen overlaps.
Parts:
- R27: footprint Resistor_SMD:R_0603_1608Metric -> Resistor_SMD:R_0805_2012Metric
Changed lines of the file:
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@@
 			)
 		)
-		(property "Footprint" "Resistor_SMD:R_0603_1608Metric"
+		(property "Footprint" "Resistor_SMD:R_0805_2012Metric"
 			(at 241.808 123.19 90)
 			(effects
